Commit message: Upload my modified robot arm project

File: ROS_WS/src/adi_robotarm/urdf/adi_robotarm.urdf (robot description, URDF)
Before this commit: robot visual, 5 links, 4 joints
Links:
- link column_link: mass 0.314159 -> 0.235619; geometry collision cylinder length=0.12 radius=0.035; visual cylinder length=0.12 radius=0.025
- link end_effector_link: mass 0.0282743 -> 0.037699; geometry collision cylinder length=0.12 radius=0.02; visual cylinder length=0.12 radius=0.01
- link lower_arm_link: mass 0.388772 -> 0.106029; geometry collision cylinder length=0.15 radius=0.025; visual cylinder length=0.15 radius=0.015
- link upper_arm_link: mass 0.69115 -> 0.175929; geometry collision cylinder length=0.14 radius=0.03; visual cylinder length=0.14 radius=0.02
Joints:
- joint base_joint: origin xyz=0 0 0.08 -> xyz=0 0 0.05
- joint elbow_joint: origin xyz=0 0 0.55 -> xyz=0 0 0.14
- joint shoulder_joint: origin xyz=0 0 0.13 -> xyz=0 0 0.12
- joint wrist_joint: limit lower=-1.5707964 upper=1.5707964 effort=81 velocity=0.5 -> lower=-3 upper=3 effort=5 velocity=2.0; origin xyz=0 0 0.55 -> xyz=0 0 0.15

Commit message: Update robot arm URDF to small endeffektor

File: ROS_WS/src/adi_robotarm/urdf/adi_robotarm.urdf (robot description, URDF)
Before this commit: robot visual, 5 links, 4 joints
Links:
- link end_effector_link: geometry collision cylinder length=0.01 radius=0.01; visual cylinder length=0.01 radius=0.01
