Commit message: servo controller exists

File: ROS_WS/src/moveit_3dof/urdf/robotarm.urdf (robot description, URDF)
Before this commit: robot robotarm, 4 links, 3 joints
Links:
- link base_link: mass 10 -> None
- link column_link: mass 0.235619 -> None
- link lower_arm_link: mass 0.106029 -> None
- link upper_arm_link: mass 0.175929 -> None

Commit message: launch robot_start working, zwischenspeichern, keyboard control

File: ROS_WS/src/moveit_3dof/urdf/robotarm.urdf (robot description, URDF)
Before this commit: robot robotarm, 4 links, 3 joints
Joints:
- joint base_joint: limit lower=-0.78539819 upper=0.78539819 effort=100 velocity=0.5 -> lower=-3.14159265 upper=3.14159265 effort=100 velocity=0.5
- joint elbow_joint: limit lower=-1.5707964 upper=1.5707964 effort=81 velocity=0.5 -> lower=-0.69813170 upper=2.44346095 effort=81 velocity=0.5; origin xyz=0 0 0.14 -> xyz=-0.025 0 0.14
- joint shoulder_joint: limit lower=-1.5707964 upper=1.5707964 effort=81 velocity=0.5 -> lower=-0.52359878 upper=1.39626340 effort=81 velocity=0.5

Commit message: encoder working

File: ROS_WS/src/moveit_3dof/urdf/robotarm.urdf (robot description, URDF)
Before this commit: robot robotarm, 4 links, 3 joints
Joints:
- joint base_joint: limit lower=-3.14159265 upper=3.14159265 effort=100 velocity=0.5 -> lower=-3.0 upper=3.0 effort=100 velocity=0.5

Commit message: moving works but directions wrong

File: ROS_WS/src/moveit_3dof/urdf/robotarm.urdf (robot description, URDF)
Before this commit: robot robotarm, 4 links, 3 joints
Links:
- added link tool_tip_link; collision sphere radius=0.012; visual sphere radius=0.01
Joints:
- added joint tool_tip_fixed_joint: type fixed, parent lower_arm_link, child tool_tip_link, origin xyz=0 0 0.15 rpy=0 0 0
