Commit message: moveit kriegt keine nachrichten

File: ROS_WS/src/robotarm_software/urdf/robotarm.urdf (robot description, URDF)
Before this commit: robot robotarm, 5 links, 4 joints
Joints:
- joint base_joint: limit lower=-3.0 upper=3.0 effort=100 velocity=0.5 -> lower=-3.14159265 upper=3.14159265 effort=100 velocity=0.30
- joint elbow_joint: limit lower=-0.69813170 upper=2.44346095 effort=81 velocity=0.5 -> lower=-0.69813170 upper=2.44346095 effort=81 velocity=0.22
- joint shoulder_joint: limit lower=-0.52359878 upper=1.39626340 effort=81 velocity=0.5 -> lower=-0.52359878 upper=1.39626340 effort=81 velocity=0.18
